Commit message: add sensors rf

File: husky_description/urdf/husky_macro.urdf.xacro (robot description, xacro)
@@ -81,4 +81,10 @@
       <parent link="${prefix}base_link" />
       <child link="${prefix}imu_link" />
+    </joint>
+    <link name="${prefix}imu_sensor" />
+    <joint name="${prefix}sensor_joint" type="fixed" >
+      <origin xyz="0 0 0" rpy="0 3.14159265 -1.57079633" />
+      <parent link="${prefix}imu_link" />
+      <child link="${prefix}imu_sensor" />
     </joint>
     <!-- GPS Link-->

File: husky_description/urdf/pic4ser.urdf.xacro (robot description, xacro)
@@ -3,9 +3,12 @@
     <xacro:include filename="$(find realsense2_description)/urdf/_d435i.urdf.xacro" />
     <xacro:include filename="$(find realsense2_description)/urdf/_d455.urdf.xacro" />
-    <xacro:sensor_d435i parent="base_link" name="camera_left" >
+    <!-- <xacro:sensor_d435i parent="base_link" name="camera_left" >
         <origin xyz="0.06 0.28 0.625" rpy="0 0 0.26" />
     </xacro:sensor_d435i>
     <xacro:sensor_d435i parent="base_link" name="camera_right" >
         <origin xyz="0.06 -0.28 0.625" rpy="0 0 -0.26" />
+    </xacro:sensor_d435i> -->
+    <xacro:sensor_d435i parent="base_link" name="camera_top_front" >
+        <origin xyz="0.045 0 0.578" rpy="0 0 0" />
     </xacro:sensor_d435i>
     <xacro:sensor_d455 parent="top_plate_front_link" name="camera_front" >
