Commit message: add prism for laser tracker

File: husky_description/urdf/pic4ser.urdf.xacro (robot description, xacro)
@@ -9,9 +9,15 @@
         <origin xyz="0.06 -0.28 0.625" rpy="0 0 -0.26" />
     </xacro:sensor_d435i> -->
-    <xacro:sensor_d435i parent="base_link" name="camera_top_front" >
+    <xacro:sensor_d455 parent="base_link" name="camera_top_front">
         <origin xyz="0.045 0 0.578" rpy="0 0 0" />
-    </xacro:sensor_d435i>
-    <xacro:sensor_d455 parent="top_plate_front_link" name="camera_front" >
+    </xacro:sensor_d455>
+    <!-- <xacro:sensor_d455 parent="top_plate_front_link" name="camera_front">
         <origin xyz="0.006 0 0.002" rpy="0 0 0" />
-    </xacro:sensor_d455>
+    </xacro:sensor_d455> -->
+    <link name="prism" />
+    <joint name="prism_joint" type="fixed">
+        <child link="prism" />
+        <parent link="top_plate_rear_link" />
+        <origin xyz="0.06 0 0.15" rpy="0 0 0" />
+    </joint>
 </robot>
